File: Circuit/ESP_Module.sch (EAGLE design)
At the start: 15 parts, among them U1 AMS1117-3.3, X2 ESP-12

Commit message: init cad design, schematics update
Parts:
- removed R3: 4.7K, SparkFun-Resistors:RESISTOR1206
- added POWER: SWITCH_SPDT_SLIDE, AutoPark:SWITCH_SPDT_SLIDE
- added R1: 1K, SparkFun-Resistors:RESISTOR1206
- R2: value 1K -> 4.7K
Connections:
- new net N$2: BATTERY.+, POWER.S
- net GND: now also R2.1; no longer R3.1
- net GPIO15: now also R2.2; no longer R3.2
- net RXD: now also R1.2; no longer R2.2
- net USB_RX: now also R1.1; no longer R2.1
- net VBAT: now also POWER.O; no longer BATTERY.+
Other:
- note removed: "RESET"
- moved on the sheet: BATTERY, R2
Changed lines of the file:
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@@
 <layer number="59" name="tCarbon" color="7" fill="1" visible="no" active="no"/>
 <layer number="60" name="bCarbon" color="7" fill="1" visible="no" active="no"/>
+<layer number="88" name="SimResults" color="9" fill="1" visible="yes" active="yes"/>
+<layer number="89" name="SimProbes" color="9" fill="1" visible="yes" active="yes"/>
 <layer number="90" name="Modules" color="7" fill="1" visible="yes" active="yes"/>
 <layer number="91" name="Nets" color="2" fill="1" visible="yes" active="yes"/>
@@
 <part name="U$1" library="microbuilder" deviceset="VBAT" device=""/>
 <part name="RN1" library="AutoPark" deviceset="CAY16-750J4LF" device="" value="10K"/>
-<part name="R3" library="SparkFun-Resistors" library_urn="urn:adsk.eagle:library:532" deviceset="RESISTOR" device="1206" package3d_urn="urn:adsk.eagle:package:39654/1" value="4.7K"/>
-<part name="R2" library="SparkFun-Resistors" library_urn="urn:adsk.eagle:library:532" deviceset="RESISTOR" device="1206" package3d_urn="urn:adsk.eagle:package:39654/1" value="1K"/>
+<part name="R2" library="SparkFun-Resistors" library_urn="urn:adsk.eagle:library:532" deviceset="RESISTOR" device="1206" package3d_urn="urn:adsk.eagle:package:39654/1" value="4.7K"/>
+<part name="R1" library="SparkFun-Resistors" library_urn="urn:adsk.eagle:library:532" deviceset="RESISTOR" device="1206" package3d_urn="urn:adsk.eagle:package:39654/1" value="1K"/>
 <part name="JP1" library="pinhead" library_urn="urn:adsk.eagle:library:325" deviceset="PINHD-1X10" device="" package3d_urn="urn:adsk.eagle:package:22406/2"/>
 <part name="JP2" library="pinhead" library_urn="urn:adsk.eagle:library:325" deviceset="PINHD-1X10" device="" package3d_urn="urn:adsk.eagle:package:22406/2"/>
@@
 <part name="PRGM" library="AutoPark" deviceset="PUSHBUTTON" device="" package3d_urn="urn:adsk.eagle:package:40165/1"/>
 <part name="U$6" library="microbuilder" deviceset="3.3V" device=""/>
+<part name="POWER" library="AutoPark" deviceset="SWITCH_SPDT_SLIDE" device=""/>
 </parts>
 <sheets>
@@
 <wire x1="142.24" y1="96.52" x2="142.24" y2="121.92" width="0.1524" layer="94" style="shortdash"/>
 <wire x1="142.24" y1="121.92" x2="111.76" y2="121.92" width="0.1524" layer="94" style="shortdash"/>
-<text x="119.38" y="170.18" size="1.778" layer="94">RESET</text>
 <wire x1="142.24" y1="121.92" x2="142.24" y2="175.26" width="0.1524" layer="94" style="shortdash"/>
 <wire x1="256.54" y1="96.52" x2="142.24" y2="96.52" width="0.1524" layer="94" style="shortdash"/>
@@
 <attribute name="VALUE" x="73.66" y="27.432" size="1.778" layer="96" font="vector" align="top-center"/>
 </instance>
-<instance part="BATTERY" gate="G$1" x="15.24" y="152.4" rot="R270">
-<attribute name="NAME" x="19.558" y="152.4" size="1.778" layer="95" font="vector" rot="R270" align="bottom-center"/>
-<attribute name="VALUE" x="10.922" y="152.4" size="1.778" layer="96" font="vector" rot="R270" align="top-center"/>
-</instance>
-<instance part="GND1" gate="1" x="15.24" y="144.78">
-<attribute name="VALUE" x="12.7" y="142.24" size="1.778" layer="96"/>
-</instance>
-<instance part="U$1" gate="G$1" x="15.24" y="160.02">
-<attribute name="VALUE" x="13.716" y="161.036" size="1.27" layer="96"/>
+<instance part="BATTERY" gate="G$1" x="124.46" y="142.24" rot="R270">
+<attribute name="NAME" x="128.778" y="142.24" size="1.778" layer="95" font="vector" rot="R270" align="bottom-center"/>
+<attribute name="VALUE" x="120.142" y="142.24" size="1.778" layer="96" font="vector" rot="R270" align="top-center"/>
+</instance>
+<instance part="GND1" gate="1" x="124.46" y="134.62">
+<attribute name="VALUE" x="121.92" y="132.08" size="1.778" layer="96"/>
+</instance>
+<instance part="U$1" gate="G$1" x="124.46" y="165.1">
+<attribute name="VALUE" x="122.936" y="166.116" size="1.27" layer="96"/>
 </instance>
 <instance part="RN1" gate="G$1" x="88.9" y="45.72" rot="R180">
@@
 <attribute name="VALUE" x="95.51396875" y="61.4746" size="2.54331875" layer="96" rot="R180"/>
 </instance>
-<instance part="R3" gate="G$1" x="119.38" y="99.06" rot="R90">
+<instance part="R2" gate="G$1" x="119.38" y="99.06" rot="R90">
 <attribute name="NAME" x="117.856" y="99.06" size="1.778" layer="95" font="vector" rot="R90" align="bottom-center"/>
 <attribute name="VALUE" x="120.904" y="99.06" size="1.778" layer="96" font="vector" rot="R90" align="top-center"/>
 </instance>
-<instance part="R2" gate="G$1" x="83.82" y="86.36" rot="R180">
+<instance part="R1" gate="G$1" x="83.82" y="86.36" rot="R180">
 <attribute name="NAME" x="83.82" y="84.836" size="1.778" layer="95" font="vector" rot="R180" align="bottom-center"/>
 <attribute name="VALUE" x="83.82" y="87.884" size="1.778" layer="96" font="vector" rot="R180" align="top-center"/>
@@
 <instance part="U$6" gate="G$1" x="99.06" y="40.64">
 <attribute name="VALUE" x="97.536" y="41.656" size="1.27" layer="96"/>
+</instance>
+<instance part="POWER" gate="G$1" x="119.38" y="154.94">
+<attribute name="NAME" x="120.65" y="157.988" size="1.778" layer="95" font="vector" align="bottom-center"/>
+<attribute name="VALUE" x="140.716" y="156.718" size="1.778" layer="96" font="vector" align="top-center"/>
 </instance>
 </instances>
@@
 <pinref part="GND2" gate="1" pin="GND"/>
 <wire x1="119.38" y1="91.44" x2="119.38" y2="93.98" width="0.1524" layer="91"/>
-<pinref part="R3" gate="G$1" pin="1"/>
+<pinref part="R2" gate="G$1" pin="1"/>
 </segment>
 <segment>
@@
 <net name="VBAT" class="0">
 <segment>
-<pinref part="BATTERY" gate="G$1" pin="+"/>
-<pinref part="U$1" gate="G$1" pin="VBAT"/>
-</segment>
-<segment>
 <pinref part="JP1" gate="A" pin="9"/>
 <wire x1="170.18" y1="60.96" x2="149.86" y2="60.96" width="0.1524" layer="91"/>
@@
 <wire x1="220.98" y1="60.96" x2="200.66" y2="60.96" width="0.1524" layer="91"/>
 <label x="200.66" y="60.96" size="1.778" layer="95"/>
+</segment>
+<segment>
+<pinref part="POWER" gate="G$1" pin="O"/>
+<pinref part="U$1" gate="G$1" pin="VBAT"/>
+<wire x1="124.46" y1="162.56" x2="124.46" y2="157.48" width="0.1524" layer="91"/>
 </segment>
 </net>
@@
 <wire x1="119.38" y1="104.14" x2="119.38" y2="116.84" width="0.1524" layer="91"/>
 <label x="119.38" y="106.68" size="1.778" layer="95" rot="R90"/>
-<pinref part="R3" gate="G$1" pin="2"/>
+<pinref part="R2" gate="G$1" pin="2"/>
 </segment>
 <segment>
@@
 <wire x1="78.74" y1="86.36" x2="60.96" y2="86.36" width="0.1524" layer="91"/>
 <label x="66.04" y="86.36" size="1.778" layer="95"/>
-<pinref part="R2" gate="G$1" pin="2"/>
+<pinref part="R1" gate="G$1" pin="2"/>
 </segment>
 <segment>
@@
 <wire x1="99.06" y1="86.36" x2="99.06" y2="101.6" width="0.1524" layer="91"/>
 <label x="99.06" y="91.44" size="1.778" layer="95" rot="R90"/>
-<pinref part="R2" gate="G$1" pin="1"/>
+<pinref part="R1" gate="G$1" pin="1"/>
 <wire x1="88.9" y1="86.36" x2="99.06" y2="86.36" width="0.1524" layer="91"/>
 </segment>
@@
 </segment>
 </net>
+<net name="N$2" class="0">
+<segment>
+<pinref part="BATTERY" gate="G$1" pin="+"/>
+<pinref part="POWER" gate="G$1" pin="S"/>
+<wire x1="124.46" y1="152.4" x2="124.46" y2="147.32" width="0.1524" layer="91"/>
+</segment>
+</net>
