File: Circuit/ESP_Module_No_Battery.sch (EAGLE design)
At the start: 16 parts, among them U1 AMS1117-3.3, X2 ESP-12

Commit message: ESP Module V1
Parts:
- removed BATTERY: BATTERY, AutoPark:BATTERY
- added J1: TERMINAL, AutoPark:TERMINAL
Connections:
- net GND: now also J1.2; no longer BATTERY.-
- net N$1: now also J1.1; no longer BATTERY.+
Changed lines of the file:
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@@
 <part name="U1" library="AutoPark" deviceset="AMS1117-3.3" device=""/>
 <part name="RESET" library="AutoPark" deviceset="PUSHBUTTON" device="" package3d_urn="urn:adsk.eagle:package:40165/1"/>
-<part name="BATTERY" library="AutoPark" deviceset="BATTERY" device=""/>
 <part name="GND1" library="supply1" library_urn="urn:adsk.eagle:library:371" deviceset="GND" device=""/>
 <part name="U$1" library="microbuilder" deviceset="VBAT" device=""/>
@@
 <part name="U$5" library="microbuilder" deviceset="VBAT" device=""/>
 <part name="POWER" library="AutoPark" deviceset="SWITCH_SPDT_SLIDE" device=""/>
+<part name="J1" library="AutoPark" deviceset="TERMINAL" device="" package3d_urn="urn:adsk.eagle:package:220531/3"/>
 </parts>
 <sheets>
@@
 <attribute name="VALUE" x="73.66" y="27.432" size="1.778" layer="96" font="vector" align="top-center"/>
 </instance>
-<instance part="BATTERY" gate="G$1" x="124.46" y="142.24" rot="R270">
-<attribute name="NAME" x="128.778" y="142.24" size="1.778" layer="95" font="vector" rot="R270" align="bottom-center"/>
-<attribute name="VALUE" x="120.142" y="142.24" size="1.778" layer="96" font="vector" rot="R270" align="top-center"/>
-</instance>
 <instance part="GND1" gate="1" x="124.46" y="134.62">
 <attribute name="VALUE" x="121.92" y="132.08" size="1.778" layer="96"/>
@@
 <attribute name="NAME" x="123.19" y="160.528" size="1.778" layer="95" font="vector" align="bottom-center"/>
 <attribute name="VALUE" x="120.396" y="151.638" size="1.778" layer="96" font="vector" align="top-center"/>
+</instance>
+<instance part="J1" gate="G$1" x="160.02" y="137.16" rot="R180">
+<attribute name="NAME" x="162.56" y="144.78" size="1.778" layer="95" rot="R180"/>
+<attribute name="VALUE" x="162.56" y="147.32" size="1.778" layer="96" rot="R180"/>
 </instance>
 </instances>
@@
 </segment>
 <segment>
-<pinref part="BATTERY" gate="G$1" pin="-"/>
-<pinref part="GND1" gate="1" pin="GND"/>
-</segment>
-<segment>
 <pinref part="JP1" gate="A" pin="10"/>
 <wire x1="170.18" y1="58.42" x2="149.86" y2="58.42" width="0.1524" layer="91"/>
@@
 <pinref part="GND4" gate="1" pin="GND"/>
 <wire x1="58.42" y1="48.26" x2="58.42" y2="43.18" width="0.1524" layer="91"/>
+</segment>
+<segment>
+<pinref part="J1" gate="G$1" pin="2"/>
+<wire x1="149.86" y1="134.62" x2="149.86" y2="137.16" width="0.1524" layer="91"/>
+<pinref part="GND1" gate="1" pin="GND"/>
+<wire x1="149.86" y1="137.16" x2="124.46" y2="137.16" width="0.1524" layer="91"/>
 </segment>
 </net>
@@
 <net name="N$1" class="0">
 <segment>
-<pinref part="BATTERY" gate="G$1" pin="+"/>
-<wire x1="124.46" y1="147.32" x2="124.46" y2="149.86" width="0.1524" layer="91"/>
-<wire x1="124.46" y1="149.86" x2="132.08" y2="149.86" width="0.1524" layer="91"/>
 <pinref part="POWER" gate="G$1" pin="O"/>
-<wire x1="132.08" y1="149.86" x2="132.08" y2="157.48" width="0.1524" layer="91"/>
 <wire x1="132.08" y1="157.48" x2="124.46" y2="157.48" width="0.1524" layer="91"/>
-</segment>
-</net>
+<pinref part="J1" gate="G$1" pin="1"/>
+<wire x1="149.86" y1="139.7" x2="132.08" y2="139.7" width="0.1524" layer="91"/>
+<wire x1="132.08" y1="139.7" x2="132.08" y2="157.48" width="0.1524" layer="91"/>
+</segment>
+</net>
